File: Hardware/KiCad/Perf/MB/Backup/Motherboard.sch (KiCad schematic (older format))
At the start: 61 parts, among them P1 Power input, P2 CONN_01X09, P3 CONN_01X05, P4 CONN_01X08, P5 CONN_02X03, P6 CONN_02X20, P7 CONN_02X20, P8 CONN_01X04, U1 STM32F100ZE, U2 LM29237-3.3, U3 SN74LVCC4245A, U4 24LC256, Y1 24MHz

Commit message: sdfghjkl
sdfghjklø
Parts:
- removed C18: 1µF, symbol CP1_Small
- removed C19: 10nF, symbol CP1_Small
- R?: renamed from R2; value 4,7k -> R
- R?: renamed from R3; value 4,7k -> R
- renumbered C17 to C4, C5 to C?, C7 to C?, C8 to C?, C9 to C?, C10 to C?, C11 to C?, C12 to C?, C13 to C?, C14 to C?, C15 to C?, C16 to C?, D1 to D?, D2 to D?, D3 to D?, D4 to D?, D5 to D?, D6 to D?, D7 to D?, D8 to D?, D9 to D?, D10 to D?, D11 to D?, D12 to D?, P2 to P?, P3 to P?, P8 to P?, P6 to P?, P7 to P?, P5 to P?, P4 to P?, R4 to R?, R5 to R?, R6 to R?, R7 to R?, R8 to R?, R9 to R?, R10 to R?, R11 to R?, R14 to R?, R15 to R?, R16 to R?, R17 to R?, R12 to R?, R13 to R?, U3 to U?, U4 to U?
Connections:
- net +3V3: no longer U1.106 (NC), U1.31 (Vref-), U1.33 (Vdda)
- net GND: now also P?.1 (P1); no longer P?.9 (P9), U1.138 (BOOT0)
- net TIM 2 CH 1: now also U?.3 (A1); no longer P?.28 (P28)
- net TIM 2 CH 2: now also U?.4 (A2); no longer P?.30 (P30)
- net TIM 2 CH 3: now also U?.5 (A3); no longer P?.32 (P32)
- net TIM 2 CH 4: now also U?.6 (A4); no longer P?.34 (P34)
- net TIM 3 CH 1: now also P?.20 (P20), U?.7 (A5); no longer U?.10 (A8)
- net TIM 3 CH 2: now also P?.22 (P22), U?.8 (A6); no longer U?.9 (A7)
- net TIM 3 CH 3: now also P?.24 (P24), U?.9 (A7); no longer U?.8 (A6)
- net TIM 3 CH 4: now also P?.26 (P26), U?.10 (A8); no longer U?.7 (A5)
- net TIM 4 CH 1: now also P?.28 (P28); no longer U?.6 (A4)
- net TIM 4 CH 2: now also P?.30 (P30); no longer U?.5 (A3)
- net TIM 4 CH 3: now also P?.32 (P32); no longer U?.4 (A2)
- net TIM 4 CH 4: now also P?.34 (P34); no longer U?.3 (A1)
- net at U1.23 (OSC_IN): now also C1.1, Y1.1; no longer R1.1
- net at U1.24 (OSC_OUT): now also R1.1
- net at P?.5 (P5), U?.18 (B4): now also R?.2; no longer R?.2
- new net: P?.9 (P9), R?.2, U?.14 (B8)
- new net: P?.8 (P8), R?.2, U?.15 (B7)
- new net: P?.7 (P7), R?.2, U?.16 (B6)
- new net: P?.6 (P6), R?.2, U?.17 (B5)
- new net: P?.4 (P4), R?.2, U?.19 (B3)
- new net: P?.3 (P3), R?.2, U?.20 (B2)
- new net: P?.2 (P2), R?.2, U?.21 (B1)
- now unconnected: U1.6 (VBAT)
Other:
- moved on the sheet: C1, C2, R1, Y1
